File: Hakari_Kicad/Hakari_Kicad.kicad_sch (KiCad schematic)
At the start: 21 parts, among them J1 FASE_A/B_ML, J2 FASE_A/B_ML, U2 MP6500, U3 MP6500

Commit message: Hakari PCB
Parts:
- removed J2: FASE_A/B_ML, symbol Connector_Generic:Conn_01x04
- removed R1, R9: 220K, symbol Device:R
- removed R10: 10K, symbol Device:R
- removed U1: (no value), Footprint:NUCLEO_H533, symbol LIB_Nucleos:Nucleo_STM32H533
- removed U2, U3: MP6500, Footprint:MP6500, symbol MOTORES_DRIVERS:MP6500
- added C10, C11, C12, C13, C14, C15, C30, C31, C34, C35, C39, C41, C44, C8: 100nF, Capacitor_SMD:C_0603_1608Metric_Pad1.08x0.95mm_HandSolder, symbol Device:C
- added C16: 4.7uF, Capacitor_SMD:C_0603_1608Metric_Pad1.08x0.95mm_HandSolder, symbol Device:C
- added C17, C32, C33: 1uF, Capacitor_SMD:C_0603_1608Metric_Pad1.08x0.95mm_HandSolder, symbol Device:C
- added C18, C19, C21, C23: 100nF, Capacitor_SMD:C_0805_2012Metric_Pad1.18x1.45mm_HandSolder, symbol Device:C
- added C20, C22: 220nF, Capacitor_SMD:C_0805_2012Metric_Pad1.18x1.45mm_HandSolder, symbol Device:C
- added C24: 10nF, Capacitor_SMD:C_0603_1608Metric_Pad1.08x0.95mm_HandSolder, symbol Device:C
- added C29: 10uF, Capacitor_Tantalum_SMD:CP_EIA-6032-15_Kemet-U_HandSolder, symbol Device:C_Polarized
- added C37: 100uF, Capacitor_Tantalum_SMD:CP_EIA-6032-15_Kemet-U_HandSolder, symbol Device:C_Polarized
- added C7, C9: 20pF, Capacitor_SMD:C_0603_1608Metric_Pad1.08x0.95mm_HandSolder, symbol Device:C
- added D10, D2, D3, D4, D5, D6, D7: LED, LED_SMD:LED_1206_3216Metric_Pad1.42x1.75mm_HandSolder, symbol Device:LED
- added H10, H11, H12, H5, H6, H7, H8, H9: MountingHole_Pad, MountingHole:MountingHole_2.2mm_M2_ISO14580_Pad, symbol Mechanical:MountingHole_Pad
- added J11: XT30_BATT, Connector_AMASS:AMASS_XT30U-F_1x02_P5.0mm_Vertical, symbol Micromouse_Library:Conector_XT30
- added J13: SQJ951EP, Package_SO:PowerPAK_SO-8_Dual, symbol Micromouse_Library:SQJ951EP-T1_BE3
- added J15, J16: (no value), Footprint:AS5145_Mod, symbol Micromouse_Library:CONN_5_PIN
- added J2: (no value), Footprint:usb_C_stm32, symbol Micromouse_Library:USB_C_SW_UART_CONECTOR
- added J3: ML, Connector_Molex:Molex_KK-254_AE-6410-04A_1x04_P2.54mm_Vertical, symbol Connector_Generic:Conn_01x04
- added J4, J5: (no value), Connector_PinHeader_2.54mm:PinHeader_1x05_P2.54mm_Vertical, symbol Micromouse_Library:CONN_5_PIN
- added J6: IR_TX, Footprint:CONN_SMD_01X04_IR, symbol Connector_Generic:Conn_01x04
- added J7: IR_RX, Footprint:CONN_SMD_01X04_IR, symbol Connector_Generic:Conn_01x04
- added J8: VCC_IR, Footprint:CONN_SMD_01X03_IR, symbol Connector_Generic:Conn_01x03
- added JP1, JP2: Jumper_2_Open, Jumper:SolderJumper-2_P1.3mm_Open_RoundedPad1.0x1.5mm, symbol Jumper:Jumper_2_Open
- added L1: 4.7uH, Inductor_SMD:L_Wuerth_HCM-7050, symbol Device:L
- added R11, R12, R13, R14, R17, R18, R56: 220, Resistor_SMD:R_0805_2012Metric_Pad1.20x1.40mm_HandSolder, symbol Device:R
- added R15: 82k, Resistor_SMD:R_0805_2012Metric_Pad1.20x1.40mm_HandSolder, symbol Device:R
- added R16: 39K, Resistor_SMD:R_0805_2012Metric_Pad1.20x1.40mm_HandSolder, symbol Device:R
- added R19, R24: 220k, Resistor_SMD:R_0805_2012Metric_Pad1.20x1.40mm_HandSolder, symbol Device:R
- added R20, R22, R57: 100k, Resistor_SMD:R_0805_2012Metric_Pad1.20x1.40mm_HandSolder, symbol Device:R
- added R21, R23: 18k, Resistor_SMD:R_0805_2012Metric_Pad1.20x1.40mm_HandSolder, symbol Device:R
- added R58, R60: 10K, Resistor_SMD:R_0805_2012Metric_Pad1.20x1.40mm_HandSolder, symbol Device:R
- added R59: 44K, Resistor_SMD:R_0805_2012Metric_Pad1.20x1.40mm_HandSolder, symbol Device:R
- added R61, R62: 10k, Resistor_SMD:R_0603_1608Metric_Pad0.98x0.95mm_HandSolder, symbol Device:R
- added SW1, SW2, SW3, SW4, SW6: SW_Push, Button_Switch_SMD:SW_Push_SPST_NO_Alps_SKRK, symbol Switch:SW_Push
- added SW5: SW_Push_SPDT, Button_Switch_SMD:SW_SPDT_PCM12, symbol Switch:SW_Push_SPDT
- added U1: (no value), Footprint:IRM-V838, symbol LIB_Componentes:IRM-V838
- added U2: (no value), Package_QFP:LQFP-64_10x10mm_P0.5mm, symbol Micromouse_Library:STM32F401RCT6
- added U25: CN3903, Package_SO:HSOP-8-1EP_3.9x4.9mm_P1.27mm_EP2.41x3.1mm, symbol Micromouse_Library:CN3903
- added U26: ME6211C33_regulador, Package_TO_SOT_SMD:SOT-23-5_HandSoldering, symbol Micromouse_Library:ME6211C33_regulador
- added U27, U28: MT6701CT, Package_SO:SO-8_3.9x4.9mm_P1.27mm, symbol Sensor_Magnetic:MT6701CT
- added U3: MPU6500, Package_DFN_QFN:QFN-24-1EP_3x3mm_P0.4mm_EP1.75x1.6mm, symbol Micromouse_Library:MPU6500
- added U4, U5: MP6500, Footprint:MP6500, symbol MOTORES_DRIVERS:MP6500
- added Y1: Crystal_GND24, Crystal:Crystal_SMD_3225-4Pin_3.2x2.5mm, symbol Device:Crystal_GND24
- C1, C4: value 100nF -> 10nF; footprint Capacitor_SMD:C_0805_2012Metric_Pad1.18x1.45mm_HandSolder -> Capacitor_SMD:C_0603_1608Metric_Pad1.08x0.95mm_HandSolder
- C2, C6: value 1uF -> 10nF; footprint Capacitor_SMD:C_0805_2012Metric_Pad1.18x1.45mm_HandSolder -> Capacitor_SMD:C_0603_1608Metric_Pad1.08x0.95mm_HandSolder
- C3: value 0.22uF -> 10nF; footprint Capacitor_SMD:C_0805_2012Metric_Pad1.18x1.45mm_HandSolder -> Capacitor_SMD:C_0603_1608Metric_Pad1.08x0.95mm_HandSolder
- C5: value 0.22uF -> 4.7uF; footprint Capacitor_SMD:C_0805_2012Metric_Pad1.18x1.45mm_HandSolder -> Capacitor_SMD:C_0603_1608Metric_Pad1.08x0.95mm_HandSolder
- J1: value FASE_A/B_ML -> MR; footprint (none) -> Connector_Molex:Molex_KK-254_AE-6410-04A_1x04_P2.54mm_Vertical
- R2, R8: value 1.5K -> 10K; footprint (none) -> Resistor_SMD:R_0805_2012Metric_Pad1.20x1.40mm_HandSolder
- R3: footprint (none) -> Resistor_SMD:R_0805_2012Metric_Pad1.20x1.40mm_HandSolder
- R4, R7: value 100K -> 10K; footprint (none) -> Resistor_SMD:R_0805_2012Metric_Pad1.20x1.40mm_HandSolder
- R5: value 20K -> 100; footprint (none) -> Resistor_SMD:R_0805_2012Metric_Pad1.20x1.40mm_HandSolder
- R6: value 20K -> 10K; footprint (none) -> Resistor_SMD:R_0805_2012Metric_Pad1.20x1.40mm_HandSolder
Connections:
- net SLEEP_ML is gone; now on net GND: R3.2
- net DIR_ML: now also U2.59 (PB7), U5.1 (DIR)
- net GND: now also C1.2, C2.2, C4.2, C6.2, R6.2, R8.2, C10.2, C11.2, C12.2, C13.2, C14.2, C15.2, C16.2, C17.2, C20.2, C22.2, C24.2, C29.2, C30.2, C32.2, C33.2, C35.2, C37.2, C44.2, C7.2, C8.2, C9.2, H5.1, H6.1, H7.1, H8.1, J11.1 (GND), J2.1 (GND), J2.12 (GND), J2.13 (SHIELD), J4.1, J5.5, J8.2 (Pin_2), R11.2, R12.2, R13.2, R14.2, R16.2, R17.2, R18.2, R19.2, R21.2, R23.2, R24.2, R56.2, R60.1, SW1.2, SW5.2 (B), U1.1 (GND), U1.4 (GND), U2.12 (VSSA/VREF---), U2.18 (VSS), U2.31 (VSS), U2.47 (VSS), U2.63 (VSS), U25.4 (GND), U25.9 (EPAD), U26.2 (VSS), U3.18 (GND), U3.20 (RESV), U3.25 (EPAD), U4.12 (GND), U4.20 (GND), U4.24 (GND), U4.25 (PAD), U4.4 (AGND), U4.8 (GND), U5.12 (GND), U5.20 (GND), U5.24 (GND), U5.25 (PAD), U5.4 (AGND), U5.8 (GND), Y1.2 (G), Y1.4 (G); no longer R4.2
- net STEP_ML: now also U2.58 (PB6), U5.13 (STEP)
- net +3.3V: now reaches C6.1
- net +3.3V: now also R2.1, R4.1, R5.1, C10.1, C11.1, C12.1, C13.1, C14.1, C15.1, C16.1, C17.1, C33.1, J2.11 (VCC), J2.2 (VCC), J4.2, J5.4, J8.3 (Pin_3), SW2.1, SW3.1, SW4.1, SW6.1, U2.1 (VBAT), U2.13 (VDDA/VREF++), U2.19 (VDD), U2.32 (VDD), U2.48 (VDD), U2.64 (VDD), U26.5 (VOUT), U3.13 (VDD), U3.8 (VDDIO)
- net BOTON_C: now reaches R8.1
- net BOTON_C: now also C24.1, SW6.2, U2.29 (PB10)
- net BOTON_B: now reaches C3.1
- net BOTON_B: now also R6.1, SW3.2, U2.28 (PB2/BOOT1)
- net BOOT0: now reaches C4.1
- net BOOT0: now also R7.1, SW4.2, U2.60 (BOOT0)
- net at R5.2: now also U1.2 (VCC); no longer R4.1
- net BOTON_A: now reaches R3.1
- net BOTON_A: now also C2.1, SW2.2, U2.27 (PB1); no longer R2.2
- net at J1.4 (Pin_4): now also U4.11 (BOUT2)
- net NRST: now reaches C1.1
- net NRST: now also R2.2, SW1.1, U2.7 (NRST)
- net at J1.2 (Pin_2): now also U4.23 (AOUT1)
- net at J1.1 (Pin_1): now also U4.21 (AOUT2)
- net at J1.3 (Pin_3): now also U4.9 (BOUT1)
- net at C5.1: now also U2.30 (VCAP1)
- new net: JP2.2 (B), R62.1, U28.2 (MODE)
- new net: D5.1 (K), R14.1
- new net: C21.1, U5.16 (CP1)
- new net: C21.2, U5.15 (CP2)
- new net: C31.2, L1.1, U25.3 (SW)
- new net: JP1.2 (B), R61.1, U27.2 (MODE)
- new net: C23.2, U5.14 (VCP)
- new net: C31.1, U25.1 (BST)
- new net: R58.2, U25.7 (EN)
- new net: C18.1, U4.16 (CP1)
- new net: C18.2, U4.15 (CP2)
- new net: D3.1 (K), R12.1
- new net: R24.1, U5.5 (ROSC)
- new net: D4.1 (K), R13.1
- new net: R20.1, U4.3 (ISET)
- new net: R20.2, R21.1
- new net: D6.1 (K), R17.1
- new net: R19.1, U4.5 (ROSC)
- new net: D7.1 (K), R18.1
- new net: J3.4 (Pin_4), U5.11 (BOUT2)
- new net: C22.1, U5.17 (VG)
- new net: J3.1 (Pin_1), U5.21 (AOUT2)
- new net: J3.2 (Pin_2), U5.23 (AOUT1)
- new net: R22.1, U5.3 (ISET)
- new net: J3.3 (Pin_3), U5.9 (BOUT1)
- new net: D10.1 (K), R56.1
- new net: C20.1, U4.17 (VG)
- new net: J13.2 (G1), J13.4 (G2), R57.2, SW5.1 (A)
- new net: R22.2, R23.1
- new net: D2.1 (K), R11.1
- new net: J11.2 (VCC), J13.1 (S1), J13.3 (S2), R57.1
- new net: C19.2, U4.14 (VCP)
- new net: C8.1, U3.10 (REGOUT)
- new net +5V: C32.1, C34.1, C35.1, C37.1, J8.1 (Pin_1), L1.2, R59.2, U26.1 (VIN), U26.3 (CE)
- new net DIR_MR: U2.57 (PB5), U4.1 (DIR)
- new net ENABLE: U2.2 (PC13), U4.18 (~ENBL), U5.18 (~ENBL)
- new net ENCA_ML: J4.3, U2.14 (PA0)
- new net ENCA_ML_CONN: J15.3, U27.6 (A)
- new net ENCA_MR: J5.3, U2.50 (PA15)
- new net ENCA_MR_CONN: J16.3, U28.6 (A)
- new net ENCB_ML: J4.4, U2.15 (PA1)
- new net ENCB_ML_CONN: J15.4, U27.7 (B)
- new net ENCB_MR: J5.2, U2.55 (PB3)
- new net ENCB_MR_CONN: J16.4, U28.7 (B)
- new net ENCC_ML: J4.5, U2.16 (PA2)
- new net ENCC_ML_CONN: J15.5, U27.8 (Z)
- new net ENCC_MR: J5.1, U2.54 (PD2)
- new net ENCC_MR_CONN: J16.5, U28.8 (Z)
- new net FN: C34.2, R59.1, R60.2, U25.5 (FB)
- new net GNDA_CONN: C39.2, H10.1, H9.1, J15.1, R61.2, U27.4 (GND)
- new net GNDB_CONN: C41.2, H11.1, H12.1, J16.1, R62.2, U28.4 (GND)
- new net IR1_RX: J7.4 (Pin_4), U2.20 (PA4)
- new net IR1_TX: J6.4 (Pin_4), U2.8 (PC0)
- new net IR2_RX: J7.3 (Pin_3), U2.21 (PA5)
- new net IR2_TX: J6.3 (Pin_3), U2.9 (PC1)
- new net IR3_RX: J7.2 (Pin_2), U2.22 (PA6)
- new net IR3_TX: J6.2 (Pin_2), U2.10 (PC2)
- new net IR4_RX: J7.1 (Pin_1), U2.23 (PA7)
- new net IR4_TX: J6.1 (Pin_1), U2.11 (PC3)
- new net IR_36KHZ: R4.2, U1.3 (OUT), U2.17 (PA3)
- new net LEDA: D2.2 (A), U2.38 (PC7)
- new net LEDB: D3.2 (A), U2.37 (PC6)
- new net LEDC: D4.2 (A), U2.36 (PB15)
- new net LEDD: D5.2 (A), U2.35 (PB14)
- new net LEDE: D6.2 (A), U2.34 (PB13)
- new net LEDF: D7.2 (A), U2.33 (PB12)
- new net MISO: U2.52 (PC11), U3.9 (ADO/SDO)
- new net MOSI: U2.53 (PC12), U3.24 (SDA/SDI)
- new net MS1: U2.61 (PB8), U4.7 (MS1), U5.7 (MS1)
- new net MS2: U2.62 (PB9), U4.6 (MS2), U5.6 (MS2)
- new net OSC_A: C7.1, U2.5 (PH0/OSC_IN), Y1.1
- new net OSC_B: C9.1, U2.6 (PH1/OSC_OUT), Y1.3
- new net RX: J2.10 (RX), J2.3 (RX), U2.43 (PA10)
- new net SCK: U2.51 (PC10), U3.23 (SCL/SCLK)
- new net SLEEP: U2.3 (PC14-OSC32_IN), U4.19 (~SLEEP), U5.19 (~SLEEP)
- new net SS: U2.45 (PA12), U3.22 (nCS)
- new net STEP_MR: U2.56 (PB4), U4.13 (STEP)
- new net SWCLK: J2.5 (SWCLK), J2.8 (SWCLK), U2.49 (PA14)
- new net SWDIO: J2.6 (SWDIO), J2.7 (SWDIO), U2.46 (PA13)
- new net TX: J2.4 (TX), J2.9 (TX), U2.42 (PA9)
- new net VCCA_CONN: C39.1, J15.2, JP1.1 (A), U27.1 (VDD)
- new net VCCB_CONN: C41.1, J16.2, JP2.1 (A), U28.1 (VDD)
- new net VIN: C19.1, C23.1, C29.1, C30.1, D10.2 (A), J13.5 (D1), J13.6 (D2), R15.1, R58.1, U25.2 (VIN), U4.10 (VIN), U4.22 (VIN), U5.10 (VIN), U5.22 (VIN)
- new net VOLTAGE_BATT: C44.1, R15.2, R16.1, U2.26 (PB0)
- no-connect marks 0 -> 12
Other:
- note added: "MOTORES MP6500"
- note removed: "Imax=71K/Rset Imax=0.6 Rset=120K"
