File: IndaV1_Kicad/IndaV1_Kicad.kicad_pcb (KiCad board)
At the start: 2 copper layers, 88 x 98.5 mm, 145 parts, among them J1 Encoder_D_Conn, J10 IR4_CONN_, J11 MOTOR_FAN, J12 Conn_01x05_Pin, J13 Conn_01x05_Pin, J14 MOTOR_ML, J15 MOTOR_MR, J16 Conn_DATOS, J17 LIPO, J18 jumper, J2 Encoder_I_Conn, J3 IR1_TX_RX_Conn, J4 IR2_TX_RX_Conn, J5 IR3_TX_RX_Conn, J6 IR4_TX_RX_Conn, J7 IR1_CONN_, J8 IR2_CONN_, J9 IR3_CONN_, Q1 AO3400A, Q2 AO3400A, Q3 AO3400A, Q4 AO3400A, Q5 AO3400A, SW1 BTN, SW2 BTN, SW3 BTN, SW4 BTN, U1 STM32F405RGT6, U2 AD8418, U3 AD8418, U4 MP6551GQB-P, U5 MP6551GQB-P, U6 MPU6500, U7 CN3903, U8 AMS1117-5.0, Y1 Crystal_GND24

Commit message: Linealizado sensores con valores obtenidos
Other:
- board text added: "106.176mm"
- board text added: "110cm"
- board text added: "121.295mm"
- board text added: "125cm"
- board text added: "136.414mm"
- board text added: "140cm"
- board text added: "151.533mm"
- board text added: "155cm"
- board text added: "166.653mm"
- board text added: "170cm"
- board text added: "181.772mm"
- board text added: "185cm"
- board text added: "196.891mm"
- board text added: "200cm"
- board text added: "212.01mm"
- board text added: "215cm"
- board text added: "227.129mm"
- board text added: "230cm"
- board text added: "242.247mm"
- board text added: "245cm"
- board text added: "257.367mm"
- board text added: "260cm"
- board text added: "275cm"
- board text added: "290cm"
- board text added: "30.5809mm"
- board text added: "305cm"
- board text added: "320cm"
- board text added: "335cm"
- board text added: "45.6929"
- board text added: "60.8191mm"
- board text added: "75.938mm"
- board text added: "91.057mm"
